File: Seeed/Adafruit-FONA-800-GSM-Breakout1.brd (EAGLE design)
At the start: 100 x 80 mm, 43 parts, among them CN2 JSTPH, IC1 74VHCT125PW, Q1 DTC143ZUAT106, SW1 KMR2, U1 SIM800H/L, U2 MCP73831T-2ACI/OT, X2 MicroB, X6 SIM_LOCKAMPHENOL

Commit message: Edit Lonet
Parts:
- removed FID1, FID2, FID3, FID4, FID5: FIDUCIAL"", microbuilder:FIDUCIAL_1MM
- removed U$33, U$34: MOUNTINGHOLE2.5, microbuilder:MOUNTINGHOLE_2.5_PLATED
- moved JP3 103.0 mm to (32.9, 15.0)
- moved D6 93.7 mm to (9.40, 1.40)
- moved TP1 92.7 mm to (32.5, 4.45)
- moved ADC 89.4 mm to (32.0, 2.16)
- moved C9 88.4 mm to (18.9, 7.87), flipped to the bottom, turned to 270 degrees
- moved D2 86.3 mm to (14.9, 3.30), turned to 90 degrees
- moved PWM 81.9 mm to (35.2, 10.8)
- moved D4 79.1 mm to (18.4, 22.2)
- moved Q1 77.1 mm to (2.41, 8.89)
- moved D5 70.6 mm to (2.16, 21.8)
- moved D3 68.7 mm to (9.91, 22.1)
- moved SW1 62.2 mm to (6.60, 21.8)
- moved IC1 17.0 mm to (31.0, 19.3)
- moved R4 3.76 mm to (4.45, 13.6)
- moved R5 3.58 mm to (4.19, 18.4)
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Routing:
- net GND: track 88.5 -> 307.9 mm, vias 2 -> 6
- net RXD_5V: track 0.00 -> 131.5 mm, vias 0 -> 3
- net VCCIO: track 0.00 -> 114.7 mm, vias 0 -> 2
- net TXD_5V: track 0.00 -> 83.5 mm, vias 0 -> 5
- net VBAT: track 41.6 -> 98.6 mm, vias 2 -> 3
- net PWM: track 0.00 -> 51.9 mm, vias 0 -> 2
- net N$16: track 0.00 -> 41.0 mm, vias 0 -> 2
- net PWRSTAT_5V: track 0.00 -> 40.8 mm, vias 0 -> 2
- net PWRSTAT: track 0.00 -> 36.6 mm, vias 0 -> 2
- net SIMCLK: track 0.00 -> 24.6 mm, vias 0 -> 1
- net SIMDATA: track 0.00 -> 23.7 mm, vias 0 -> 1
- net 1.8V: track 0.00 -> 20.9 mm, vias 0 -> 1
- net UART_TXD: track 0.00 -> 20.5 mm, vias 0 -> 2
- net SIMRST: track 0.00 -> 20.4 mm
- net PWRKEY: track 0.00 -> 17.5 mm, vias 0 -> 2
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