File: LoNet/LoNet800L.sch (EAGLE design)
At the start: 36 parts, among them K1 3.3X3.3MM, Q4 BC846BW, Q5 BC846BW, U1 SIM800L

Commit message: Change LoNet 800L with RFM69 and batter recharger
Connections:
- net H_DTR: now also U$1.GPIO17/GEN0
- net PWR: now also U$1.GPIO4/GCKL
- net RI: now also U$1.GPIO18
- net R_DIO0: now also U$1.GEN/6GPIO25
- net R_DIO2: now also U$1.GEN4/GPIO23
- net R_NSS: now also U$1.!CE0!/GPIO8
- net R_RESET: now also U$1.GEN5/GPIO24
- net R_SCK: now also U$1.GPIO11/SCLK
Changed lines of the file:
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@@
 <setting verticaltext="up"/>
 </settings>
-<grid distance="50" unitdist="mil" unit="mil" style="lines" multiple="1" display="no" altdistance="0.01" altunitdist="inch" altunit="inch"/>
+<grid distance="0.1" unitdist="inch" unit="inch" style="lines" multiple="1" display="no" altdistance="0.01" altunitdist="inch" altunit="inch"/>
 <layers>
 <layer number="1" name="Top" color="4" fill="1" visible="no" active="no"/>
@@
 <label x="838.2" y="106.68" size="1.778" layer="95"/>
 </segment>
+<segment>
+<pinref part="U$1" gate="G$1" pin="GPIO4/GCKL"/>
+<wire x1="1031.24" y1="205.74" x2="1018.54" y2="205.74" width="0.1524" layer="91"/>
+<label x="1018.54" y="205.74" size="1.778" layer="95"/>
+</segment>
 </net>
 <net name="VBAT" class="0">
@@
 <label x="985.52" y="212.09" size="1.27" layer="95" xref="yes"/>
 </segment>
+<segment>
+<pinref part="U$1" gate="G$1" pin="GPIO18"/>
+<wire x1="1079.5" y1="200.66" x2="1089.66" y2="200.66" width="0.1524" layer="91"/>
+<label x="1082.04" y="200.66" size="1.778" layer="95"/>
+</segment>
 </net>
 <net name="ANT" class="0">
@@
 <label x="838.2" y="111.76" size="1.778" layer="95"/>
 </segment>
+<segment>
+<pinref part="U$1" gate="G$1" pin="GPIO17/GEN0"/>
+<wire x1="1031.24" y1="200.66" x2="1018.54" y2="200.66" width="0.1524" layer="91"/>
+<label x="1018.54" y="200.66" size="1.778" layer="95"/>
+</segment>
 </net>
 <net name="VIO" class="0">
@@
 <label x="1078.23" y="118.11" size="1.778" layer="95"/>
 </segment>
+<segment>
+<pinref part="U$1" gate="G$1" pin="GEN4/GPIO23"/>
+<wire x1="1079.5" y1="195.58" x2="1092.2" y2="195.58" width="0.1524" layer="91"/>
+<label x="1079.5" y="195.58" size="1.778" layer="95"/>
+</segment>
 </net>
 <net name="R_DIO0" class="0">
@@
 <label x="1019.81" y="102.87" size="1.778" layer="95"/>
 </segment>
+<segment>
+<pinref part="U$1" gate="G$1" pin="GEN/6GPIO25"/>
+<wire x1="1079.5" y1="187.96" x2="1092.2" y2="187.96" width="0.1524" layer="91"/>
+<label x="1079.5" y="187.96" size="1.778" layer="95"/>
+</segment>
 </net>
 <net name="R_RESET" class="0">
@@
 <label x="1019.81" y="118.11" size="1.778" layer="95"/>
 </segment>
+<segment>
+<pinref part="U$1" gate="G$1" pin="GEN5/GPIO24"/>
+<wire x1="1079.5" y1="193.04" x2="1092.2" y2="193.04" width="0.1524" layer="91"/>
+<label x="1079.5" y="193.04" size="1.778" layer="95"/>
+</segment>
 </net>
 <net name="R_NSS" class="0">
@@
 <label x="1019.81" y="115.57" size="1.778" layer="95"/>
 </segment>
+<segment>
+<pinref part="U$1" gate="G$1" pin="!CE0!/GPIO8"/>
+<wire x1="1079.5" y1="185.42" x2="1092.2" y2="185.42" width="0.1524" layer="91"/>
+<label x="1079.5" y="185.42" size="1.778" layer="95"/>
+</segment>
 </net>
 <net name="R_SCK" class="0">
@@
 <label x="1019.81" y="113.03" size="1.778" layer="95"/>
 </segment>
-</net>
+<segment>
+<pinref part="U$1" gate="G$1" pin="GPIO11/SCLK"/>
+<wire x1="1031.24" y1="185.42" x2="1018.54" y2="185.42" width="0.1524" layer="91"/>
+<label x="1018.54" y="185.42" size="1.778" layer="95"/>
+</segment>
+</net>
